Commit message: Divided ROS Packages adn Updated README

File: simulation/simulation_rviz/urdf/manipulator.urdf (robot description, URDF)
Before this commit: robot manipulator, 6 links, 5 joints
Links:
- link link_0: geometry collision mesh filename=package://simulation_rviz/meshes/link_0.STL; visual mesh filename=package://simulation_rviz/meshes/link_0.STL
- link link_1: geometry collision mesh filename=package://simulation_rviz/meshes/link_1.STL; visual mesh filename=package://simulation_rviz/meshes/link_1.STL
- link link_2: geometry collision mesh filename=package://simulation_rviz/meshes/link_2.STL; visual mesh filename=package://simulation_rviz/meshes/link_2.STL
- link link_3: geometry collision mesh filename=package://simulation_rviz/meshes/link_3.STL; visual mesh filename=package://simulation_rviz/meshes/link_3.STL
