Commit message: Add new model to package, update publishing scripts

File: 3_simulation_rviz/urdf/manipulator.urdf (robot description, URDF)
Before this commit: robot manipulator, 6 links, 5 joints
Links:
- removed link link_0
- removed link link_4
- added link base_link, mass 0.0896; collision mesh filename=package://simulation_rviz/meshes/base_link.STL; visual mesh filename=package://simulation_rviz/meshes/base_link.STL
- added link claw_left, mass 0.013642; collision mesh filename=package://simulation_rviz/meshes/claw_left.STL; visual mesh filename=package://simulation_rviz/meshes/claw_left.STL
- added link claw_right, mass 0.043225; collision mesh filename=package://simulation_rviz/meshes/claw_right.STL; visual mesh filename=package://simulation_rviz/meshes/claw_right.STL
- link link_1: mass 0.021123 -> 0.024846
- link link_2: mass 0.016936 -> 0.01633
- link link_3: mass 0.0089186 -> 0.019923
Joints:
- added joint joint_5: type revolute, parent link_3, child claw_left, origin xyz=0.079643 0.0231993 -0.020398 rpy=0 0.2 0, axis 0 0 1, limit lower=0 upper=0.9 effort=1.0 velocity=1.0
- joint dummy_joint: child link_0 -> base_link
- joint joint_1: limit lower=0.0 upper=3.14159265359 effort=1.0 velocity=1.0 -> lower=-1.57 upper=1.57 effort=1.0 velocity=1.0; origin xyz=0.0029256 -5.3727E-05 0.1232 rpy=0 0 0.011222 -> xyz=-0.0030196 0.046937 0.0635 rpy=0 0 0; parent link_0 -> base_link
- joint joint_2: axis 0 0 1 -> 0 1 0; limit lower=0.0 upper=3.14159265359 effort=1.0 velocity=0.0 -> lower=-1.26 upper=1.26 effort=1.0 velocity=1.0; origin xyz=-0.00029839 0.01004 0.039318 rpy=1.5708 0.0098142 0 -> xyz=0.0010394 -0.0095198 0.034407 rpy=0 0 0
- joint joint_3: axis 0 0 1 -> 0 1 0; limit lower=0.0 upper=3.14159265359 effort=1.0 velocity=0.0 -> lower=-1.87 upper=0.80 effort=1.0 velocity=1.0; origin xyz=0.1199 0 0.01365 rpy=0 0 -1.57079632679 -> xyz=-0.00063851 0.011696 0.072593 rpy=0 0 0
- joint joint_4: axis (none) -> 0 0 -1; child link_4 -> claw_right; limit (none) -> lower=0 upper=0.9 effort=1.0 velocity=1.0; origin xyz=0.0899 0.002 0.0037 rpy=0 0 0 -> xyz=0.091729 -0.0080548 -0.011749 rpy=0 0.2 0; type fixed -> revolute

Commit message: Update model to work within 0 to 180 deg

File: 3_simulation_rviz/urdf/manipulator.urdf (robot description, URDF)
Before this commit: robot manipulator, 7 links, 6 joints
Links:
- link claw_left: mass 0.013642 -> 0.013641
- link claw_right: mass 0.043225 -> 0.013225
Joints:
- joint joint_1: limit lower=-1.57 upper=1.57 effort=1.0 velocity=1.0 -> lower=0 upper=3.14 effort=1.0 velocity=1.0
- joint joint_2: axis 0 1 0 -> 0 -1 0; limit lower=-1.26 upper=1.26 effort=1.0 velocity=1.0 -> lower=0 upper=3.14 effort=1 velocity=1; origin xyz=0.0010394 -0.0095198 0.034407 rpy=0 0 0 -> xyz=0.00031511 -0.0095653 0.034407 rpy=0 0 0
- joint joint_3: axis 0 1 0 -> 0 -1 0; limit lower=-1.87 upper=0.80 effort=1.0 velocity=1.0 -> lower=0 upper=3.14 effort=1 velocity=1; origin xyz=-0.00063851 0.011696 0.072593 rpy=0 0 0 -> xyz=0.071531 0.011279 -0.0041348 rpy=0 0 0
- joint joint_4: axis 0 0 -1 -> -1 0 0; limit lower=0 upper=0.9 effort=1.0 velocity=1.0 -> lower=0 upper=0.8 effort=1.0 velocity=1.0; origin xyz=0.091729 -0.0080548 -0.011749 rpy=0 0.2 0 -> xyz=0.020925 -0.013767 -0.090331 rpy=0 0 0
- joint joint_5: axis 0 0 1 -> 1 0 0; limit lower=0 upper=0.9 effort=1.0 velocity=1.0 -> lower=0 upper=0.8 effort=1.0 velocity=1.0; origin xyz=0.079643 0.0231993 -0.020398 rpy=0 0.2 0 -> xyz=0.0091023 0.0182709 -0.090512 rpy=0 0 0
