Commit message: [ Fixing Bugs ] : Collision error persists

File: 3_simulation_gazebo/urdf/manipulator.urdf (robot description, URDF)
Before this commit: robot manipulator, 7 links, 6 joints
Links:
- link base_link: geometry visual mesh filename=package://simulation_gazebo/meshes/base_link.STL
- link claw_left: geometry visual mesh filename=package://simulation_gazebo/meshes/claw_left.STL
- link claw_right: geometry visual mesh filename=package://simulation_gazebo/meshes/claw_right.STL
- link link_1: geometry visual mesh filename=package://simulation_gazebo/meshes/link_1.STL
- link link_2: geometry visual mesh filename=package://simulation_gazebo/meshes/link_2.STL
- link link_3: geometry visual mesh filename=package://simulation_gazebo/meshes/link_3.STL

Commit message: [Minor Tweaks] :Adds position controllers instead of joint trajectory controller, problem of vibration remains unresolved

File: 3_simulation_gazebo/urdf/manipulator.urdf (robot description, URDF)
Before this commit: robot manipulator, 7 links, 6 joints
Links:
- link base_link: geometry collision mesh filename=package://simulation_gazebo/meshes/base_link.STL; visual mesh filename=package://simulation_gazebo/meshes/base_link.STL
- link claw_right: geometry collision mesh filename=package://simulation_gazebo/meshes/claw_right.STL; visual mesh filename=package://simulation_gazebo/meshes/claw_right.STL
- link link_1: geometry collision mesh filename=package://simulation_gazebo/meshes/link_1.STL; visual mesh filename=package://simulation_gazebo/meshes/link_1.STL
- link link_2: geometry collision mesh filename=package://simulation_gazebo/meshes/link_2.STL; visual mesh filename=package://simulation_gazebo/meshes/link_2.STL
- link link_3: geometry collision mesh filename=package://simulation_gazebo/meshes/link_3.STL; visual mesh filename=package://simulation_gazebo/meshes/link_3.STL
Joints:
- joint joint_1: limit lower=0 upper=3.14 effort=1.0 velocity=1.0 -> lower=0 upper=6.28 effort=1.0 velocity=1.0
- joint joint_2: limit lower=0 upper=3.14 effort=1 velocity=1 -> lower=-3 upper=3 effort=1 velocity=1
- joint joint_4: limit lower=0 upper=0.8 effort=1.0 velocity=1.0 -> lower=-0.8 upper=0.8 effort=1.0 velocity=1.0
- joint joint_5: limit lower=0 upper=0.8 effort=1.0 velocity=1.0 -> lower=0.2 upper=0.8 effort=1.0 velocity=1.0

Commit message: [ URDF Exports ] : URDF with old config is currently attached, later will change to the new URDF

File: 3_simulation_gazebo/urdf/manipulator.urdf (robot description, URDF)
Before this commit: robot manipulator, 7 links, 6 joints
Links:
- link claw_left: geometry collision mesh filename=package://simulation_gazebo/meshes/claw_left.STL; visual mesh filename=package://simulation_gazebo/meshes/claw_left.STL
Joints:
- joint joint_1: limit lower=0 upper=6.28 effort=1.0 velocity=1.0 -> lower=0 upper=3.14 effort=1.0 velocity=1.0
- joint joint_2: limit lower=-3 upper=3 effort=1 velocity=1 -> lower=0 upper=3.14 effort=1 velocity=1
- joint joint_4: limit lower=-0.8 upper=0.8 effort=1.0 velocity=1.0 -> lower=0 upper=0.8 effort=1.0 velocity=1.0
- joint joint_5: limit lower=0.2 upper=0.8 effort=1.0 velocity=1.0 -> lower=0 upper=0.8 effort=1.0 velocity=1.0
